File: Wireless Flex Node.brd (EAGLE design)
At the start: 83.7 x 50 mm, 39 parts, among them IC2 317T, P1 2X4_HEADER, P2 2X4_HEADER

Commit message: Update Wireless Flex Node.brd
Parts:
- removed IC2: 317T, linear:TO220H
- added IC1: 317T, linear:TO220H
- added R8: 4.7k, rcl:0207/10
- moved U$8 1.26 mm to (36.1, 34.8)
- moved U$9 0.50 mm to (48.5, 33.8)
Connections:
- net N$24: now also R8.2
- net N$32: now also IC1.3; no longer IC2.3
- net N$33: now also IC1.1; no longer IC2.1
- net N$34: now also IC1.2; no longer IC2.2
- net VCC: now also R8.1
Routing:
- net N$32: track 21.1 -> 31.4 mm
- net N$24: track 17.9 -> 24.4 mm
- net N$33: track 11.2 -> 16.4 mm
- net N$34: track 21.8 -> 24.7 mm
- net VCC: track 143.3 -> 146.1 mm
- net N$30: track 9.62 -> 7.92 mm
- net N$28: track 5.86 -> 4.71 mm
- net N$26: track 5.64 -> 4.79 mm
Other:
- board text added: "."
- board text added: "or TMP36"
