File: Wireless Flex Node.sch (EAGLE design)
At the start: 39 parts, among them IC2 317T, P1 2X4_HEADER, P2 2X4_HEADER

Commit message: Update Wireless Flex Node.sch
Parts:
- removed IC2: 317T, linear:317T
- added IC1: 317T, linear:317T
- added R8: 4.7k, rcl:R-EU_0207/10
Connections:
- net N$24: now also R8.2
- net N$32: now also IC1.VI; no longer IC2.VI
- net N$33: now also IC1.ADJ; no longer IC2.ADJ
- net N$34: now also IC1.VO; no longer IC2.VO
- net VCC: now also R8.1; no longer U$9.VCC
Changed lines of the file:
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@@
 <part name="EVE" library="ForceTronics" deviceset="2PINHEADER_S" device=""/>
 <part name="N3" library="ForceTronics" deviceset="2.1MM_DC_JACK" device=""/>
-<part name="IC2" library="linear" deviceset="*317" device="T"/>
 <part name="GND10" library="supply1" deviceset="GND" device=""/>
 <part name="C4" library="rcl" deviceset="C-EU" device="050-030X075" value="100n"/>
@@
 <part name="P1" library="ForceTronics" deviceset="2X4_HEADER" device=""/>
 <part name="P2" library="ForceTronics" deviceset="2X4_HEADER" device=""/>
+<part name="IC1" library="linear" deviceset="*317" device="T"/>
+<part name="R8" library="rcl" deviceset="R-EU_" device="0207/10" value="4.7k"/>
 </parts>
 <sheets>
@@
 <instance part="GND8" gate="1" x="78.74" y="-12.7"/>
 <instance part="U$8" gate="G$1" x="152.4" y="-12.7"/>
-<instance part="U$9" gate="G$1" x="129.54" y="88.9" rot="R270"/>
+<instance part="U$9" gate="G$1" x="195.326" y="88.9" rot="R270"/>
 <instance part="IRQ" gate="G$1" x="162.56" y="38.1" rot="R270"/>
 <instance part="IRQ" gate="G$2" x="160.02" y="38.1" rot="R270"/>
@@
 <instance part="EVE" gate="G$2" x="119.38" y="-7.62" rot="R270"/>
 <instance part="N3" gate="DCJACK" x="-13.97" y="6.35" rot="R180"/>
-<instance part="IC2" gate="A1" x="12.7" y="-1.27"/>
 <instance part="GND10" gate="1" x="-7.62" y="-12.7"/>
 <instance part="C4" gate="G$1" x="0" y="-3.81" rot="R180"/>
@@
 <instance part="P2" gate="R1" x="157.48" y="109.22"/>
 <instance part="P2" gate="R2" x="142.24" y="109.22" rot="MR0"/>
+<instance part="IC1" gate="A1" x="12.954" y="-1.27"/>
+<instance part="R8" gate="G$1" x="182.88" y="83.82" rot="R90"/>
 </instances>
 <busses>
@@
 <wire x1="121.92" y1="99.06" x2="124.46" y2="99.06" width="0.1524" layer="91"/>
 <wire x1="124.46" y1="99.06" x2="124.46" y2="106.68" width="0.1524" layer="91"/>
-<pinref part="U$9" gate="G$1" pin="VCC"/>
-<wire x1="124.46" y1="86.36" x2="121.92" y2="86.36" width="0.1524" layer="91"/>
 <wire x1="121.92" y1="86.36" x2="121.92" y2="99.06" width="0.1524" layer="91"/>
 <junction x="121.92" y="99.06"/>
+<wire x1="121.92" y1="86.36" x2="175.26" y2="86.36" width="0.1524" layer="91"/>
+<wire x1="175.26" y1="86.36" x2="175.26" y2="78.74" width="0.1524" layer="91"/>
+<wire x1="190.5" y1="86.36" x2="187.96" y2="86.36" width="0.1524" layer="91"/>
+<wire x1="187.96" y1="86.36" x2="187.96" y2="78.74" width="0.1524" layer="91"/>
+<pinref part="R8" gate="G$1" pin="1"/>
+<wire x1="187.96" y1="78.74" x2="182.88" y2="78.74" width="0.1524" layer="91"/>
+<wire x1="175.26" y1="78.74" x2="182.88" y2="78.74" width="0.1524" layer="91"/>
+<junction x="182.88" y="78.74"/>
 </segment>
 <segment>
@@
 <junction x="114.3" y="101.6"/>
 <pinref part="U$9" gate="G$1" pin="GND"/>
-<wire x1="124.46" y1="91.44" x2="119.38" y2="91.44" width="0.1524" layer="91"/>
+<wire x1="190.246" y1="91.44" x2="119.38" y2="91.44" width="0.1524" layer="91"/>
 <wire x1="119.38" y1="91.44" x2="119.38" y2="101.6" width="0.1524" layer="91"/>
 <wire x1="119.38" y1="101.6" x2="114.3" y2="101.6" width="0.1524" layer="91"/>
@@
 <pinref part="DGHDFGH" gate="1" pin="ANALOG_0"/>
 <pinref part="U$9" gate="G$1" pin="DQ"/>
-<wire x1="96.52" y1="88.9" x2="124.46" y2="88.9" width="0.1524" layer="91"/>
+<wire x1="96.52" y1="88.9" x2="182.88" y2="88.9" width="0.1524" layer="91"/>
+<pinref part="R8" gate="G$1" pin="2"/>
+<wire x1="182.88" y1="88.9" x2="190.246" y2="88.9" width="0.1524" layer="91"/>
+<junction x="182.88" y="88.9"/>
 </segment>
 </net>
@@
 <segment>
 <pinref part="N3" gate="DCJACK" pin="VIN"/>
-<pinref part="IC2" gate="A1" pin="VI"/>
-<wire x1="2.54" y1="1.27" x2="0" y2="1.27" width="0.1524" layer="91"/>
+<wire x1="2.794" y1="1.27" x2="0" y2="1.27" width="0.1524" layer="91"/>
 <pinref part="C4" gate="G$1" pin="2"/>
 <wire x1="0" y1="1.27" x2="-8.89" y2="1.27" width="0.1524" layer="91"/>
 <junction x="0" y="1.27"/>
+<pinref part="IC1" gate="A1" pin="VI"/>
 </segment>
 </net>
@@
 <segment>
 <pinref part="R1" gate="G$1" pin="1"/>
-<pinref part="IC2" gate="A1" pin="ADJ"/>
-<wire x1="12.7" y1="-8.89" x2="12.7" y2="-6.35" width="0.1524" layer="91"/>
+<wire x1="12.7" y1="-8.89" x2="12.954" y2="-6.35" width="0.1524" layer="91"/>
 <pinref part="R2" gate="G$1" pin="2"/>
 <wire x1="25.4" y1="-8.89" x2="12.7" y2="-8.89" width="0.1524" layer="91"/>
@@
 <pinref part="R3" gate="G$1" pin="1"/>
 <wire x1="12.7" y1="-8.89" x2="7.62" y2="-8.89" width="0.1524" layer="91"/>
+<pinref part="IC1" gate="A1" pin="ADJ"/>
 </segment>
 </net>
 <net name="N$34" class="0">
 <segment>
-<pinref part="IC2" gate="A1" pin="VO"/>
 <pinref part="R2" gate="G$1" pin="1"/>
-<wire x1="25.4" y1="1.27" x2="22.86" y2="1.27" width="0.1524" layer="91"/>
+<wire x1="25.4" y1="1.27" x2="23.114" y2="1.27" width="0.1524" layer="91"/>
 <pinref part="PWR_JUMP" gate="G$3" pin="S"/>
 <wire x1="25.4" y1="1.27" x2="34.29" y2="1.27" width="0.1524" layer="91"/>
@@
 <wire x1="34.29" y1="1.27" x2="40.64" y2="1.27" width="0.1524" layer="91"/>
 <junction x="34.29" y="1.27"/>
-</segment>
-</net>
+<pinref part="IC1" gate="A1" pin="VO"/>
+</segment>
+</net>
