File: Wireless Flex Node SMD.sch (EAGLE design)
At the start: 31 parts, among them IC2 LM317, P1 2X4_HEADER, P2 2X4_HEADER

Commit message: Update Wireless Flex Node SMD.sch
Parts:
- removed EVE, SCL, SDA: 2PINHEADER_S, ForceTronics:2PINHEADER_S
- removed R1: 360, rcl:R-US_R1206
- removed R2: 220, rcl:R-US_R1206
- added A4, A5, D5, D7, D8: 1PINHEADER_S, ForceTronics:1PINHEADER_S
- IC2: value LM317 -> LP2985; device linear:317EMP -> ForceTronics:LP2985
Connections:
- removed net N$27: DGHDFGH.ANALOG_5, SCLG$2.S
- removed net N$29: DGHDFGH.ANALOG_4, SDAG$2.S
- removed net N$30: EVEG$1.S, U$8.EVENT
- removed net N$31: DGHDFGH.DIGITAL_5(PWM), EVEG$2.S
- removed net N$33: IC2.ADJ, R1.2, R2.1
- new net A5: D5.S, DGHDFGH.DIGITAL_5(PWM), U$8.EVENT
- net GND: now also IC2.GND; no longer R1.1
- net N$11: now also D7.S
- net N$16: now also D8.S
- net N$26: now also A5.S, DGHDFGH.ANALOG_5; no longer SCLG$1.S
- net N$28: now also A4.S, DGHDFGH.ANALOG_4; no longer SDAG$1.S
- net N$32: now also IC2.EN, IC2.IN; no longer IC2.VI
- net N$34: now also IC2.OUT; no longer IC2.VO, R2.2
Other:
- moved on the sheet: C6
Changed lines of the file:
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@@
 <part name="P+7" library="supply1" deviceset="VCC" device=""/>
 <part name="GND9" library="supply1" deviceset="GND" device=""/>
-<part name="SCL" library="ForceTronics" deviceset="2PINHEADER_S" device=""/>
-<part name="SDA" library="ForceTronics" deviceset="2PINHEADER_S" device=""/>
-<part name="EVE" library="ForceTronics" deviceset="2PINHEADER_S" device=""/>
 <part name="N3" library="ForceTronics" deviceset="2.1MM_DC_JACK" device=""/>
 <part name="GND10" library="supply1" deviceset="GND" device=""/>
@@
 <part name="LED3" library="adafruit" deviceset="LED" device="SMT1206"/>
 <part name="LED4" library="adafruit" deviceset="LED" device="SMT1206"/>
-<part name="R1" library="rcl" deviceset="R-US_" device="R1206" value="360"/>
-<part name="R2" library="rcl" deviceset="R-US_" device="R1206" value="220"/>
 <part name="R3" library="rcl" deviceset="R-US_" device="R1206" value="100k"/>
 <part name="C7" library="rcl" deviceset="C-US" device="C1206" value="10uF"/>
 <part name="C8" library="rcl" deviceset="C-US" device="C1206" value="0.1uF"/>
-<part name="IC2" library="linear" deviceset="*317" device="EMP" value="LM317"/>
 <part name="R6" library="rcl" deviceset="R-US_" device="R1206" value="220"/>
 <part name="R10" library="rcl" deviceset="R-US_" device="R1206" value="220"/>
@@
 <part name="C4" library="rcl" deviceset="C-US" device="C1206" value="0.1uF"/>
 <part name="OSC1" library="ForceTronics" deviceset="CSTCE_RESONATOR" device=""/>
+<part name="IC2" library="ForceTronics" deviceset="LP2985" device=""/>
+<part name="D5" library="ForceTronics" deviceset="1PINHEADER_S" device=""/>
+<part name="A4" library="ForceTronics" deviceset="1PINHEADER_S" device=""/>
+<part name="A5" library="ForceTronics" deviceset="1PINHEADER_S" device=""/>
+<part name="D8" library="ForceTronics" deviceset="1PINHEADER_S" device=""/>
+<part name="D7" library="ForceTronics" deviceset="1PINHEADER_S" device=""/>
 </parts>
 <sheets>
@@
 <instance part="P+7" gate="VCC" x="142.24" y="25.4"/>
 <instance part="GND9" gate="1" x="144.78" y="-17.78"/>
-<instance part="SCL" gate="G$1" x="139.7" y="-2.54" rot="R270"/>
-<instance part="SCL" gate="G$2" x="137.16" y="-2.54" rot="R270"/>
-<instance part="SDA" gate="G$1" x="132.08" y="-12.7" rot="R270"/>
-<instance part="SDA" gate="G$2" x="129.54" y="-12.7" rot="R270"/>
-<instance part="EVE" gate="G$1" x="121.92" y="-7.62" rot="R270"/>
-<instance part="EVE" gate="G$2" x="119.38" y="-7.62" rot="R270"/>
 <instance part="N3" gate="DCJACK" x="-13.97" y="6.35" rot="R180"/>
 <instance part="GND10" gate="1" x="-7.62" y="-12.7"/>
@@
 <instance part="P2" gate="R2" x="142.24" y="109.22" rot="MR0"/>
 <instance part="R9" gate="G$1" x="20.32" y="101.6" rot="R90"/>
-<instance part="C6" gate="G$1" x="0" y="-1.27"/>
+<instance part="C6" gate="G$1" x="-2.54" y="-1.27"/>
 <instance part="LED3" gate="G$1" x="34.29" y="-12.7"/>
 <instance part="LED4" gate="G$1" x="91.44" y="7.62"/>
-<instance part="R1" gate="G$1" x="12.7" y="-13.97" rot="R90"/>
-<instance part="R2" gate="G$1" x="26.67" y="-3.81" rot="R90"/>
 <instance part="R3" gate="G$1" x="78.74" y="5.08" rot="R90"/>
 <instance part="C7" gate="G$1" x="154.94" y="82.55" rot="R270"/>
 <instance part="C8" gate="G$1" x="20.32" y="43.18"/>
-<instance part="IC2" gate="A1" x="13.97" y="-1.27"/>
 <instance part="R6" gate="G$1" x="34.29" y="-3.81" rot="R90"/>
 <instance part="R10" gate="G$1" x="91.44" y="16.51" rot="R90"/>
@@
 <instance part="C4" gate="G$1" x="50.8" y="101.6" rot="R90"/>
 <instance part="OSC1" gate="G$1" x="-5.08" y="73.66"/>
+<instance part="IC2" gate="G$1" x="7.62" y="-11.43"/>
+<instance part="D5" gate="G$1" x="114.3" y="-10.16"/>
+<instance part="A4" gate="G$1" x="129.54" y="-17.78" rot="R270"/>
+<instance part="A5" gate="G$1" x="121.92" y="0" rot="R180"/>
+<instance part="D8" gate="G$1" x="99.06" y="-12.7" rot="R270"/>
+<instance part="D7" gate="G$1" x="85.09" y="21.59" rot="R180"/>
 </instances>
 <busses>
@@
 <wire x1="-8.89" y1="5.08" x2="-7.62" y2="5.08" width="0.1524" layer="91"/>
 <junction x="-7.62" y="5.08"/>
-<wire x1="0" y1="-6.35" x2="0" y2="-8.89" width="0.1524" layer="91"/>
-<wire x1="0" y1="-8.89" x2="-7.62" y2="-8.89" width="0.1524" layer="91"/>
+<wire x1="-2.54" y1="-6.35" x2="-2.54" y2="-8.89" width="0.1524" layer="91"/>
+<wire x1="-2.54" y1="-8.89" x2="-7.62" y2="-8.89" width="0.1524" layer="91"/>
 <junction x="-7.62" y="-8.89"/>
 <pinref part="C6" gate="G$1" pin="2"/>
@@
 <wire x1="34.29" y1="-19.05" x2="12.7" y2="-19.05" width="0.1524" layer="91"/>
 <pinref part="LED3" gate="G$1" pin="C"/>
-<pinref part="R1" gate="G$1" pin="1"/>
+<pinref part="IC2" gate="G$1" pin="GND"/>
+<wire x1="2.54" y1="-8.89" x2="2.54" y2="-19.05" width="0.1524" layer="91"/>
+<wire x1="2.54" y1="-19.05" x2="12.7" y2="-19.05" width="0.1524" layer="91"/>
 <junction x="12.7" y="-19.05"/>
 </segment>
@@
 <pinref part="R3" gate="G$1" pin="1"/>
 <junction x="78.74" y="0"/>
+<pinref part="D8" gate="G$1" pin="S"/>
+<wire x1="99.06" y1="0" x2="99.06" y2="-10.16" width="0.1524" layer="91"/>
+<junction x="99.06" y="0"/>
 </segment>
 </net>
@@
 <segment>
 <pinref part="U$8" gate="G$1" pin="SCL"/>
-<pinref part="SCL" gate="G$1" pin="S"/>
-<wire x1="147.32" y1="0" x2="139.7" y2="0" width="0.1524" layer="91"/>
-</segment>
-</net>
-<net name="N$27" class="0">
-<segment>
-<pinref part="SCL" gate="G$2" pin="S"/>
+<wire x1="147.32" y1="0" x2="137.16" y2="0" width="0.1524" layer="91"/>
 <wire x1="137.16" y1="0" x2="137.16" y2="76.2" width="0.1524" layer="91"/>
 <pinref part="DGHDFGH" gate="1" pin="ANALOG_5"/>
 <wire x1="137.16" y1="76.2" x2="96.52" y2="76.2" width="0.1524" layer="91"/>
+<pinref part="A5" gate="G$1" pin="S"/>
+<wire x1="124.46" y1="0" x2="137.16" y2="0" width="0.1524" layer="91"/>
+<junction x="137.16" y="0"/>
 </segment>
 </net>
@@
 <segment>
 <pinref part="U$8" gate="G$1" pin="SDA"/>
-<pinref part="SDA" gate="G$1" pin="S"/>
-<wire x1="147.32" y1="-10.16" x2="132.08" y2="-10.16" width="0.1524" layer="91"/>
-</segment>
-</net>
-<net name="N$29" class="0">
-<segment>
-<pinref part="SDA" gate="G$2" pin="S"/>
+<wire x1="147.32" y1="-10.16" x2="129.54" y2="-10.16" width="0.1524" layer="91"/>
 <wire x1="129.54" y1="-10.16" x2="129.54" y2="78.74" width="0.1524" layer="91"/>
 <pinref part="DGHDFGH" gate="1" pin="ANALOG_4"/>
 <wire x1="129.54" y1="78.74" x2="96.52" y2="78.74" width="0.1524" layer="91"/>
-</segment>
-</net>
-<net name="N$30" class="0">
-<segment>
-<pinref part="U$8" gate="G$1" pin="EVENT"/>
-<pinref part="EVE" gate="G$1" pin="S"/>
-<wire x1="147.32" y1="-5.08" x2="121.92" y2="-5.08" width="0.1524" layer="91"/>
-</segment>
-</net>
-<net name="N$31" class="0">
-<segment>
-<pinref part="EVE" gate="G$2" pin="S"/>
-<wire x1="119.38" y1="-5.08" x2="100.33" y2="-5.08" width="0.1524" layer="91"/>
+<pinref part="A4" gate="G$1" pin="S"/>
+<wire x1="129.54" y1="-15.24" x2="129.54" y2="-10.16" width="0.1524" layer="91"/>
+<junction x="129.54" y="-10.16"/>
+</segment>
+</net>
+<net name="A5" class="0">
+<segment>
 <wire x1="100.33" y1="-5.08" x2="100.33" y2="53.34" width="0.1524" layer="91"/>
 <pinref part="DGHDFGH" gate="1" pin="DIGITAL_5(PWM)"/>
 <wire x1="96.52" y1="53.34" x2="100.33" y2="53.34" width="0.1524" layer="91"/>
+<pinref part="U$8" gate="G$1" pin="EVENT"/>
+<wire x1="147.32" y1="-5.08" x2="111.76" y2="-5.08" width="0.1524" layer="91"/>
+<pinref part="D5" gate="G$1" pin="S"/>
+<wire x1="111.76" y1="-5.08" x2="100.33" y2="-5.08" width="0.1524" layer="91"/>
+<wire x1="111.76" y1="-10.16" x2="111.76" y2="-5.08" width="0.1524" layer="91"/>
+<junction x="111.76" y="-5.08"/>
 </segment>
 </net>
@@
 <segment>
 <pinref part="N3" gate="DCJACK" pin="VIN"/>
-<wire x1="3.81" y1="1.27" x2="0" y2="1.27" width="0.1524" layer="91"/>
-<pinref part="IC2" gate="A1" pin="VI"/>
 <pinref part="C6" gate="G$1" pin="1"/>
-<wire x1="0" y1="1.27" x2="-8.89" y2="1.27" width="0.1524" layer="91"/>
-<junction x="0" y="1.27"/>
-</segment>
-</net>
-<net name="N$33" class="0">
-<segment>
-<wire x1="26.67" y1="-8.89" x2="13.97" y2="-8.89" width="0.1524" layer="91"/>
-<pinref part="R1" gate="G$1" pin="2"/>
-<pinref part="R2" gate="G$1" pin="1"/>
-<pinref part="IC2" gate="A1" pin="ADJ"/>
-<wire x1="13.97" y1="-8.89" x2="12.7" y2="-8.89" width="0.1524" layer="91"/>
-<wire x1="13.97" y1="-6.35" x2="13.97" y2="-8.89" width="0.1524" layer="91"/>
-<junction x="13.97" y="-8.89"/>
+<wire x1="-2.54" y1="1.27" x2="-8.89" y2="1.27" width="0.1524" layer="91"/>
+<junction x="-2.54" y="1.27"/>
+<pinref part="IC2" gate="G$1" pin="IN"/>
+<wire x1="-2.54" y1="1.27" x2="2.54" y2="1.27" width="0.1524" layer="91"/>
+<pinref part="IC2" gate="G$1" pin="EN"/>
+<wire x1="2.54" y1="1.27" x2="2.54" y2="-3.81" width="0.1524" layer="91"/>
+<junction x="2.54" y="1.27"/>
 </segment>
 </net>
@@
 <segment>
 <pinref part="PWR_JUMP" gate="G$3" pin="S"/>
-<pinref part="IC2" gate="A1" pin="VO"/>
-<wire x1="24.13" y1="1.27" x2="26.67" y2="1.27" width="0.1524" layer="91"/>
-<pinref part="R2" gate="G$1" pin="2"/>
-<wire x1="26.67" y1="1.27" x2="34.29" y2="1.27" width="0.1524" layer="91"/>
-<junction x="26.67" y="1.27"/>
 <pinref part="R6" gate="G$1" pin="2"/>
 <wire x1="34.29" y1="1.27" x2="40.64" y2="1.27" width="0.1524" layer="91"/>
+<pinref part="IC2" gate="G$1" pin="OUT"/>
+<wire x1="30.48" y1="1.27" x2="34.29" y2="1.27" width="0.1524" layer="91"/>
 <junction x="34.29" y="1.27"/>
 </segment>
@@
 <wire x1="96.52" y1="48.26" x2="97.79" y2="48.26" width="0.1524" layer="91"/>
 <wire x1="97.79" y1="48.26" x2="97.79" y2="21.59" width="0.1524" layer="91"/>
-<wire x1="91.44" y1="21.59" x2="97.79" y2="21.59" width="0.1524" layer="91"/>
 <pinref part="R10" gate="G$1" pin="2"/>
-</segment>
-</net>
+<pinref part="D7" gate="G$1" pin="S"/>
+<wire x1="87.63" y1="21.59" x2="97.79" y2="21.59" width="0.1524" layer="91"/>
+<wire x1="87.63" y1="21.59" x2="91.44" y2="21.59" width="0.1524" layer="91"/>
+<junction x="87.63" y="21.59"/>
+</segment>
+</net>
